File: Documentacion, Especificacion y Diseño/Diagramas/Ejemplo1/Proyecto.kicad_pcb (KiCad board)
At the start: 2 copper layers, 13 parts, among them J1 Conn_01x02, U1 LM7805_TO220, U2 PIC16F886-IP, Y1 20MHz

Commit message: Idme diciendo que os parece
Parts:
- moved C2 37.6 mm to (134.0, 93.5)
- moved C3 37.6 mm to (137.8, 116.4)
- moved C4 37.6 mm to (137.8, 111.3)
- moved J1 37.6 mm to (135.2, 102.7)
- moved C1 37.6 mm to (140.3, 96.1)
- moved PickIt3 37.6 mm to (177.2, 84.7)
- moved SCLySDAyCCPySCKySDO1 37.6 mm to (136.5, 127.8)
- moved U1 37.6 mm to (140.3, 87.2)
- moved U2 37.6 mm to (150.5, 92.3)
- moved EntradasRuHuTe1 37.6 mm to (145.4, 98.6)
- moved R1 37.6 mm to (145.4, 87.8)
- moved USART1 37.6 mm to (163.2, 115.1)
- moved Y1 37.6 mm to (145.4, 116.4)
Other:
- board outline added: 59.4 x 59.2 mm
- board text added: "CCP1"
- board text added: "GM1"
- board text added: "SCK"
- board text added: "SCL"
- board text added: "SDA"
- board text added: "SDO"
- board text added: "TX"
- board text added: "V"
- board text added: "h"
- board text added: "r"
- board text added: "t"

Commit message: arreglo del circuito y documento, disenio fisico y video arq alto nivel completados
Other:
- outline, holes or cut-outs redrawn
- board text added: "ccp"
- board text added: "scl"
Changed lines of the file:
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@@
   (general
     (thickness 1.6)
-    (drawings 28)
+    (drawings 43)
     (tracks 97)
     (zones 0)
@@
     (visible_elements 7FFFFFFF)
     (pcbplotparams
-      (layerselection 0x010fc_ffffffff)
+      (layerselection 0x00000_fffffffe)
       (usegerberextensions false)
       (usegerberattributes true)
       (usegerberadvancedattributes true)
       (creategerberjobfile true)
-      (excludeedgelayer true)
+      (excludeedgelayer false)
       (linewidth 0.100000)
       (plotframeref false)
@@
       (padsonsilk false)
       (subtractmaskfromsilk false)
-      (outputformat 1)
+      (outputformat 2)
       (mirror false)
-      (drillshape 1)
+      (drillshape 2)
       (scaleselection 1)
       (outputdirectory ""))
@@
     )
   )
+  (gr_text ccp (at 141 121 90) (layer B.Cu)
+    (effects (font (size 2 2) (thickness 0.5)) (justify mirror))
+  )
+  (gr_text scl (at 136 121 90) (layer B.Cu)
+    (effects (font (size 2 2) (thickness 0.5)) (justify mirror))
+  )
+  (gr_text t (at 143 105) (layer B.Cu)
+    (effects (font (size 2 2) (thickness 0.5)) (justify mirror))
+  )
+  (gr_text r (at 143 98.5) (layer B.Cu)
+    (effects (font (size 2 2) (thickness 0.5)) (justify mirror))
+  )
+  (gr_text TX (at 167 120.5) (layer B.Cu)
+    (effects (font (size 2 2) (thickness 0.5)) (justify mirror))
+  )
+  (gr_text V (at 182 84.5 -90) (layer B.Cu)
+    (effects (font (size 2 2) (thickness 0.5)))
+  )
+  (gr_text GM1 (at 178.5 126.5) (layer B.Cu)
+    (effects (font (size 2 2) (thickness 0.5)) (justify mirror))
+  )
+  (gr_circle (center 130 133.5) (end 132 133.5) (layer Edge.Cuts) (width 0.8))
+  (gr_circle (center 182.5 132.5) (end 184.5 133) (layer Edge.Cuts) (width 0.8))
+  (gr_circle (center 130.5 81) (end 132.5 81) (layer Edge.Cuts) (width 0.8))
+  (gr_circle (center 182.5 81) (end 184.5 81) (layer Edge.Cuts) (width 0.8))
+  (gr_circle (center 130.5 81) (end 133 81) (layer Edge.Cuts) (width 0.8))
+  (gr_circle (center 130 133.5) (end 132.5 133.5) (layer Edge.Cuts) (width 0.8))
+  (gr_circle (center 182.5 132.5) (end 185 132.5) (layer Edge.Cuts) (width 0.8))
+  (gr_circle (center 182.5 81) (end 185 81) (layer Edge.Cuts) (width 0.8))
   (dimension 2.5 (width 0.15) (layer Dwgs.User)
     (gr_text "2,500 mm" (at 175.7 133.77 270) (layer Dwgs.User)
